File: Hardware/Controller_Room/Controller_Room.kicad_pcb (KiCad board)
At the start: 2 copper layers, 75.3 x 54.4 mm, 73 parts, among them IC1 RY8310, J1 Barrel_Jack_Switch, J10 Conn_01x04_Female, J2 HR911105A, J4 Conn_01x04_Female, J5 Conn_01x04_Female, J6 Conn_01x04_Female, J7 Conn_01x06_Female, J8 Conn_01x02_Female, M1 P-CHANNEL-MOSFET, M2 P-CHANNEL-MOSFET, Q1 Q_NPN_BEC, SW1 Reset, SW2 User, U1 ESP32-WROOM-32, U2 LAN8720A, U3 MAX3485, U4 ACS711xLCTR-12AB, X1 ASV-50MHz

Commit message: Add Files
Parts:
- removed C17: 100n, Capacitor_SMD:C_0402_1005Metric
- removed J1: Barrel_Jack_Switch, Techbeard:BarrelJack_10A
- removed J10: Conn_01x04_Female, Connector_PinHeader_2.54mm:PinHeader_1x04_P2.54mm_Vertical
- removed J2: HR911105A, Techbeard:HR911105A
- removed J8: Conn_01x02_Female, Connector_PinHeader_2.54mm:PinHeader_1x02_P2.54mm_Vertical
- removed M1, M2: P-CHANNEL-MOSFET, Package_SON:VSON-8_3.3x3.3mm_P0.65mm_NexFET
- removed Q1: Q_NPN_BEC, Package_TO_SOT_SMD:SOT-23
- removed R26: 100, Capacitor_SMD:C_0402_1005Metric
- added C20: 100n, Capacitor_SMD:C_0402_1005Metric, B.Cu at (214.3, 115.4)
- added C21: 100n, Capacitor_SMD:C_0402_1005Metric, B.Cu at (203.0, 123.3)
- added C22: 100n, Capacitor_SMD:C_0402_1005Metric, B.Cu at (203.0, 124.4)
- added C23: 1000pF/2KV, Capacitor_SMD:C_1206_3216Metric, B.Cu at (190.4, 122.7)
- added C24: 100n, Capacitor_SMD:C_0402_1005Metric, B.Cu at (190.3, 118.7)
- added C25: 100n, Capacitor_SMD:C_0402_1005Metric, B.Cu at (192.8, 118.7)
- added C26: 1000pF/2KV, Capacitor_SMD:C_1206_3216Metric, B.Cu at (192.5, 107.6)
- added J3: HP DPS, LCSC:CONN-TH_64P-P2.54_ED64MEBGFBK, B.Cu at (190.3, 137.3)
- added L3: B1608S, LCSC:B1608S, B.Cu at (206.3, 115.4)
- added R30: 75, Resistor_SMD:R_0402_1005Metric, B.Cu at (201.0, 123.3)
- added R31: 75, Resistor_SMD:R_0402_1005Metric, B.Cu at (201.0, 124.5)
- added R32: 75, Resistor_SMD:R_0402_1005Metric, B.Cu at (190.3, 119.8)
- added R33: 75, Resistor_SMD:R_0402_1005Metric, B.Cu at (192.8, 119.8)
- added R36: 0, Capacitor_SMD:C_1206_3216Metric, B.Cu at (189.2, 107.6)
- added U5: RC01931, LCSC:RJ45-TH_RCH_RC01931, F.Cu at (190.1, 120.8)
- C1, C10, C11, C12, C13, C14, C15, C16, C18, C2, C3, C4, C5, C7, C8, C9, IC1, L1, L2, R10, R11, R12, R13, R14, R15, R16, R17, R18, R19, R2, R20, R21, R22, R23, R24, R25, R3, R6, R7, R8, U1, U2, U3, X1: moved to B.Cu
- C6: value 22u -> 10u; footprint Capacitor_SMD:CP_Elec_5x5.4 -> Capacitor_SMD:C_1206_3216Metric; moved to B.Cu
- D4: value 15V -> LED; footprint Diode_SMD:D_0402_1005Metric -> LED_SMD:LED_0402_1005Metric
- J6: footprint Connector_Phoenix_GMSTB:PhoenixContact_GMSTBA_2,5_4-G-7,62_1x04_P7.62mm_Horizontal -> LCSC:CONN-TH_4P-P7.62_DB2EVC-7.62-4P
- R1: value 1k -> 10k; moved to B.Cu
- R4: value 100k -> 22k
- R5: value 4k7 -> R; moved to B.Cu
- R9: footprint Resistor_SMD:R_0402_1005Metric -> Resistor_SMD:R_1206_3216Metric; moved to B.Cu
- U4: value ACS711xLCTR-12AB -> EL817S1(C)(TU)-F; footprint Package_SO:SOIC-8_3.9x4.9mm_P1.27mm -> LCSC:OPTO-SMD-4_L4.6-W6.5-P2.54-LS10.3-TL; moved to B.Cu
- moved H4 231.1 mm to (3.48, 11.4)
- moved H3 181.1 mm to (3.48, 3.48)
- moved J7 104.9 mm to (247.6, 124.7), turned to 180 degrees
- moved U4 99.7 mm to (246.3, 135.6)
- moved R5 97.6 mm to (245.1, 129.0), turned to 180 degrees
- moved R4 89.7 mm to (220.8, 138.2), turned to 0 degrees
- moved R17 65.5 mm to (217.7, 127.3), turned to 180 degrees
- moved R25 63.8 mm to (216.0, 123.3), turned to 0 degrees
- moved C12 63.0 mm to (217.7, 129.3), turned to 0 degrees
- moved C13 62.2 mm to (217.7, 128.3), turned to 0 degrees
- moved L2 61.3 mm to (212.1, 121.1), turned to 0 degrees
- moved C14 61.3 mm to (212.1, 122.2), turned to 180 degrees
- moved C15 61.2 mm to (212.1, 123.2), turned to 180 degrees
- moved R24 61.1 mm to (213.4, 119.9), turned to 180 degrees
- moved R22 60.8 mm to (213.4, 113.5), turned to 180 degrees
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Connections:
- C1 pad 1: VCC -> +12V
- C12 pad 1: +3V3 -> Net-(U2-VDDCR)
- C13 pad 1: +3V3 -> Net-(U2-VDDCR)
- C2 pad 1: VCC -> +12V
- D4 pad 1: VCC -> GND
- D4 pad 2: Net-(D4-Pad2) -> Net-(D4-A)
- IC1 pad 4: unconnected-(IC1-Pad4) -> +12V
- IC1 pad 5: VCC -> +12V
- J6 pad 2: A -> B
- J6 pad 3: B -> A
- R1 pad 1: VCC -> +VSW
- R4 pad 1: Net-(D4-Pad2) -> +12V
- R4 pad 2: GND -> /HP DPS High/PRESENT#
- R5 pad 1: PowerSW -> +3V3
- R5 pad 2: Net-(Q1-Pad1) -> Net-(U4-AN)
- R6 pad 1: VCC -> +12V
- R6 pad 2: Net-(M2-Pad4) -> Net-(D4-A)
- U1 pad 14: Net-(J8-Pad1) -> RS485_RO
- U1 pad 23: Net-(J8-Pad2) -> SCL
- U1 pad 24: WS28_Out -> SDA
- U1 pad 26: SCL -> RS485_DI
- U1 pad 29: SDA -> unconnected-(U1-IO5-Pad29)
- U1 pad 5: PowerMES -> unconnected-(U1-SENSOR_VN-Pad5)
- U1 pad 6: IO34 -> unconnected-(U1-IO34-Pad6)
- U1 pad 7: IO35 -> unconnected-(U1-IO35-Pad7)
- U1 pad 8: IO32 -> RS485_DE
- U1 pad 9: IO33 -> RS485_RE
- U2 pad 6: +3V3 -> Net-(U2-VDDCR)
- U3 pad 1: unconnected-(U3-Pad1) -> RS485_RO
- U3 pad 2: +3V3 -> RS485_RE
- U3 pad 3: +3V3 -> RS485_DE
- U3 pad 4: WS28_Out -> RS485_DI
- U4 pad 1: +VSW -> Net-(U4-AN)
- U4 pad 2: +VSW -> PowerSW
- U4 pad 3: Net-(M2-Pad5) -> GND
- U4 pad 4: Net-(M2-Pad5) -> /HP DPS High/PSON#
Routing:
- net +3V3: track 295.1 -> 27.0 mm, vias 11 -> 16
- net PowerMES: track 71.8 -> 0.00 mm
- net StateLED: track 63.2 -> 0.00 mm
- net PowerSW: track 62.8 -> 11.0 mm
- net IO26_RXD1: track 36.4 -> 1.09 mm, vias 2 -> 1
- net IO25_RXD0: track 35.5 -> 1.08 mm, vias 2 -> 1
- net EN: track 42.3 -> 8.93 mm
- net GND: track 48.1 -> 19.6 mm, vias 39 -> 38
- net Net-(U2-LED1/REGOFF): track 4.24 -> 31.9 mm, vias 0 -> 2
- net +12V: track 0.00 -> 27.3 mm, vias 0 -> 3
- net Net-(L3-TX+): track 0.00 -> 21.1 mm
- net WS28_Out: track 20.8 -> 0.00 mm
- net ETHLEDYel: track 22.4 -> 1.67 mm
- net +VSW: track 0.00 -> 20.0 mm
- net Net-(U2-LED2/nINTSEL): track 3.22 -> 23.1 mm, vias 0 -> 2
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- added copper zone on In2.Cu, net +3V3
- added copper zone on B.Cu, net +VSW
- added copper zone on In1.Cu, net GND
- removed copper zone on F.Cu, net +3V3
- removed copper zone on F.Cu, net +VSW
- removed copper zone on B.Cu, net GND
- removed copper zone on F.Cu, net Net-(IC1-SW)
- removed copper zone on F.Cu, net Net-(J1-Pad1)
- removed copper zone on F.Cu, net Net-(M2-Pad5)
- removed copper zone on F.Cu, net VCC
Other:
- board size 75.3 x 54.4 mm -> 119 x 39 mm
- copper layers 2 -> 4
- board text added: "Mia Depta, Valentin Fischer, LeoDj"
- board text removed: "A"
- board text removed: "B"
- board text removed: "Gnd"
- board text removed: "Mia Depta, Pascal Schubert, Nico Martin, Valentin Fischer"
- board text removed: "Naschkatzen"
- board text removed: "Vcc"
