File: Hardware/Controller_Room/Controller_Room.kicad_sch (KiCad schematic)
At the start: 73 parts, among them IC1 RY8310, J1 Barrel_Jack_Switch, J10 Conn_01x04_Female, J4 Conn_01x04_Female, J5 Conn_01x04_Female, J6 Conn_01x04_Female, J7 Conn_01x06_Female, J8 Conn_01x02_Female, M1 P-CHANNEL-MOSFET, M2 P-CHANNEL-MOSFET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

Commit message: fix Bodges in Schematic
Parts:
- J2: value (none) -> HR911105A; footprint (none) -> Techbeard:HR911105A
- J6: footprint (none) -> Connector_Phoenix_GMSTB:PhoenixContact_GMSTBA_2,5_4-G-7,62_1x04_P7.62mm_Horizontal
- X1: footprint (none) -> Oscillator:Oscillator_SMD_Abracon_ASE-4Pin_3.2x2.5mm
Connections:
- net +3.3VA: now also J2.4 (TCT), J2.5 (RCT)
- net +3V3: no longer C12.1, C13.1, U2.6 (VDDCR)
- net GND: no longer J2.4 (TCT), J2.5 (RCT)
- net VCC: now also IC1.4 (EN)
- new net: C12.1, C13.1, U2.6 (VDDCR)
- no-connect marks 8 -> 7
Other:
- moved on the sheet: J6

Commit message: Add Files
Parts:
- removed C17: 100n, Capacitor_SMD:C_0402_1005Metric, symbol Device:C
- removed C6: 22u, Capacitor_SMD:CP_Elec_5x5.4, symbol Device:C_Polarized
- removed D4: 15V, Diode_SMD:D_0402_1005Metric, symbol Device:D_Zener
- removed J1: Barrel_Jack_Switch, Techbeard:BarrelJack_10A, symbol Connector:Barrel_Jack_Switch
- removed J10: Conn_01x04_Female, Connector_PinHeader_2.54mm:PinHeader_1x04_P2.54mm_Vertical, symbol Connector:Conn_01x04_Female
- removed J2: HR911105A, Techbeard:HR911105A, symbol Techbeard:HR911105A
- removed J8: Conn_01x02_Female, Connector_PinHeader_2.54mm:PinHeader_1x02_P2.54mm_Vertical, symbol Connector:Conn_01x02_Female
- removed M1, M2: P-CHANNEL-MOSFET, Package_SON:VSON-8_3.3x3.3mm_P0.65mm_NexFET, symbol Techbeard:P-CHANNEL-MOSFET
- removed Q1: Q_NPN_BEC, Package_TO_SOT_SMD:SOT-23, symbol Device:Q_NPN_BEC
- removed R26: 100, Capacitor_SMD:C_0402_1005Metric, symbol Device:R
- removed U4: ACS711xLCTR-12AB, Package_SO:SOIC-8_3.9x4.9mm_P1.27mm, symbol Sensor_Current:ACS711xLCTR-12AB
- added C6: 10u, Capacitor_SMD:C_1206_3216Metric, symbol Device:C
- added D4: LED, LED_SMD:LED_0402_1005Metric, symbol Device:LED
- added U4: EL817S1(C)(TU)-F, LCSC:OPTO-SMD-4_L4.6-W6.5-P2.54-LS10.3-TL, symbol LCSC:EL817S1(C)(TU)-F
- J6: footprint Connector_Phoenix_GMSTB:PhoenixContact_GMSTBA_2,5_4-G-7,62_1x04_P7.62mm_Horizontal -> LCSC:CONN-TH_4P-P7.62_DB2EVC-7.62-4P
- R1: value 1k -> 10k
- R4: value 100k -> 22k
- R5: value 4k7 -> R
- R9: footprint Resistor_SMD:R_0402_1005Metric -> Resistor_SMD:R_1206_3216Metric
Connections:
- net +3V3: now also R5.1, C6.1; no longer U3.2 (~{RE}), U3.3 (DE)
- net +VSW: now also R1.1
- net A: now also J6.3 (Pin_3); no longer J6.2 (Pin_2)
- net B: now also J6.2 (Pin_2); no longer J6.3 (Pin_3)
- net GND: now also C6.2, D4.1 (K), U4.3 (EM); no longer R4.2
- net PowerSW: now also U4.2 (CAT); no longer R5.1
- net SCL: now also U1.23 (IO15); no longer U1.26 (IO4)
- net SDA: now also U1.24 (IO2); no longer U1.29 (IO5)
- net at R5.2: now also U4.1 (AN)
- net at R6.2: now also D4.2 (A)
- net +12V: now reaches R4.1
- net +12V: now also C1.1, C2.1, IC1.4 (EN), IC1.5 (IN), R6.1
- net RS485_RO: now reaches U1.14 (IO12)
- net RS485_RO: now also U3.1 (RO)
- net IO32 renamed RS485_DE
- net RS485_DE: now also U3.3 (DE)
- net IO33 renamed RS485_RE
- net RS485_RE: now also U3.2 (~{RE})
- net IO34: no longer names the net of U1.6 (IO34)
- net IO35: no longer names the net of U1.7 (IO35)
- net PowerMES: no longer names the net of U1.5 (SENSOR_VN)
- removed net VCC: C1.1, C2.1, IC1.4 (EN), IC1.5 (IN), R1.1, R6.1
- net WS28_Out renamed RS485_DI
- net RS485_DI: now also U1.26 (IO4); no longer U1.24 (IO2)
- new net HP DPS High/PRESENT#: R4.2
- new net HP DPS High/PSON#: U4.4 (COL)
Other:
- added sheet Ethernet (Ethernet.kicad_sch)
- added sheet HP DPS High (hp_dps.kicad_sch)
- moved on the sheet: C1, C2, C4, C5, D1, D2, D3, IC1, L1, R1, R10, R11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
